File: GCM_powerSupply.sch (KiCad schematic (older format))
At the start: 34 parts, among them J1 Screw_Terminal_01x02, J2 Barrel_Jack_Switch, J3 Molex_1053101108, J4 Screw_Terminal_01x04, SW1 SW_SPDT, U1 TPS563201, U2 TPS563201

Commit message: Fix R0805 was 1206, change the switch
Parts:
- SW1: footprint LSSA12VB:LSSA12VB -> EG1218:EG1218
Changed lines of the file:
@@
 F 0 "SW1" H 1650 5235 50  0000 C CNN
 F 1 "SW_SPDT" H 1650 5144 50  0000 C CNN
-F 2 "LSSA12VB:LSSA12VB" H 1650 4950 50  0001 C CNN
+F 2 "EG1218:EG1218" H 1650 4950 50  0001 C CNN
 F 3 "~" H 1650 4950 50  0001 C CNN
 	1    1650 4950
